File: Page3.kicad_sch (KiCad schematic)
At the start: 19 parts, among them IC1 LEXI-R10801D-00B-00, J10 SSW-110-03-G-S, J11 SSW-110-03-G-S, J12 SSW-110-03-G-S, J13 Conn_01x14_Pin, J14 Conn_01x14_Pin, J15 Conn_01x14_Pin, J16 Conn_01x14_Pin, J17 Conn_01x14_Pin, J18 Conn_01x14_Pin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

Commit message: test1
Parts:
- removed U5: NEO-8Q, RF_GPS:ublox_NEO, symbol RF_GPS:NEO-8Q
- removed U6: MAX-M10S, RF_GPS:ublox_MAX, symbol RF_GPS:MAX-M10S
- removed U7: ZED-F9P, RF_GPS:ublox_ZED, symbol RF_GPS:ZED-F9P
- IC1: footprint LEXIR10801D00B00 -> footprints2:LEXIR10801D00B00
Connections:
- net GND: now also J10.10 (Pin_10), J11.10 (Pin_10), J12.10 (Pin_10), J5.10 (Pin_10), J9.10 (Pin_10)
- net V_INT: now reaches J9.1 (Pin_1)
- net V_INT: now also J10.1 (Pin_1), J5.1 (Pin_1)
- net CELL_GPIO5: now reaches J9.9 (Pin_9)
- net VCC: now reaches J12.1 (Pin_1)
- net VCC: now also J11.1 (Pin_1)
- net CELL_GPIO4: now reaches J5.2 (Pin_2)
- net CELL_GPIO2: now reaches J5.3 (Pin_3)
- net CELL_GPIO1: now reaches J5.4 (Pin_4)
- net SDA: now reaches J5.5 (Pin_5)
- net SCL: now reaches J5.6 (Pin_6)
- net RI: now reaches J5.7 (Pin_7)
- net RTS: now reaches J5.8 (Pin_8)
- net CTS: now reaches J5.9 (Pin_9)
- net CELL_GPIO6: now reaches J10.9 (Pin_9)
- net USB_BOOT: now reaches J11.9 (Pin_9)
Other:
- moved on the sheet: J10, J11, J12, J9
