File: LEXI-ADAM UNO SHIELD ver.01.kicad_pcb (KiCad board)
At the start: 4 copper layers, 53.3 x 68.6 mm, 84 parts, among them IC1 LEXI-R10801D-00B-00, J1 SSW-106-03-G-S, J10 SSW-110-03-G-S, J11 SSW-110-03-G-S, J12 SSW-110-03-G-S, J13 Conn_01x14_Pin, J14 Conn_01x14_Pin, J15 Conn_01x14_Pin, J16 Conn_01x14_Pin, J17 Conn_01x14_Pin, J18 Conn_01x14_Pin, J19 Conn_01x14_Pin, J2 SSW-110-03-G-S, J20 Conn_01x14_Pin, J21 Conn_01x14_Pin, J22 Conn_01x14_Pin, J23 Conn_Coaxial, J3 SSW-108-03-G-S, J4 SSW-108-03-G-S, J5 SSW-110-03-G-S, J6 MSIM-2-A, J7 Conn_Coaxial, J8 USB_C_Receptacle_USB2.0_16P, J9 SSW-110-03-G-S, SW1 B3FS-1000P, SW4 B3FS-1000P, U2 SLM37ECB800, U3 LMR51450FNDRRR, U4 TXU0204PWR, U5 NEO-8Q, U6 MAX-M10S, U7 ZED-F9P, U8 74LVC2G07GV,125

Commit message: test1
Parts:
- removed U5: NEO-8Q, RF_GPS:ublox_NEO
- removed U6: MAX-M10S, RF_GPS:ublox_MAX
- removed U7: ZED-F9P, RF_GPS:ublox_ZED
- moved J10 1.46 mm to (164.3, 89.4)
- moved J15 1.46 mm to (160.9, 72.4)
- moved J20 1.46 mm to (167.3, 72.4)
- moved J21 1.46 mm to (168.5, 72.4)
- moved J9 1.46 mm to (161.8, 89.4)
- moved J11 1.46 mm to (166.8, 89.4)
- moved J12 1.46 mm to (169.4, 89.4)
- moved J13 1.46 mm to (158.4, 72.4)
- moved J14 1.46 mm to (159.6, 72.4)
- moved J16 1.46 mm to (162.2, 72.4)
- moved J17 1.46 mm to (163.5, 72.4)
- moved J18 1.46 mm to (164.7, 72.4)
- moved J19 1.46 mm to (166.0, 72.4)
- moved J22 1.46 mm to (169.8, 72.4)
- moved J5 1.46 mm to (159.2, 89.4)
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Connections:
- IC1 pad 10: unconnected-(IC1A-RI-Pad10) -> RI
- IC1 pad 11: unconnected-(IC1A-DSR-Pad11) -> DSR
- IC1 pad 12: unconnected-(IC1A-SCL-Pad12) -> SCL
- IC1 pad 13: unconnected-(IC1A-SDA-Pad13) -> SDA
- IC1 pad 14: unconnected-(IC1A-GPIO1-Pad14) -> CELL_GPIO1
- IC1 pad 15: unconnected-(IC1A-GPIO2-Pad15) -> CELL_GPIO2
- IC1 pad 17: unconnected-(IC1A-GPIO4-Pad17) -> CELL_GPIO4
- IC1 pad 18: unconnected-(IC1A-GPIO5-Pad18) -> CELL_GPIO5
- IC1 pad 29: unconnected-(IC1A-GPIO6-Pad29) -> CELL_GPIO6
- IC1 pad 48: unconnected-(IC1A-USB_BOOT-Pad48) -> USB_BOOT
- IC1 pad 6: unconnected-(IC1A-CTS-Pad6) -> CTS
- IC1 pad 8: unconnected-(IC1A-DCD-Pad8) -> DCD
- J10 pad 1: unconnected-(J10-Pin_1-Pad1) -> V_INT
- J10 pad 10: unconnected-(J10-Pin_10-Pad10) -> GND
- J10 pad 9: unconnected-(J10-Pin_9-Pad9) -> CELL_GPIO6
- J11 pad 1: unconnected-(J11-Pin_1-Pad1) -> VCC
- J11 pad 10: unconnected-(J11-Pin_10-Pad10) -> GND
- J11 pad 9: unconnected-(J11-Pin_9-Pad9) -> USB_BOOT
- J12 pad 1: unconnected-(J12-Pin_1-Pad1) -> VCC
- J12 pad 10: unconnected-(J12-Pin_10-Pad10) -> GND
- J5 pad 1: unconnected-(J5-Pin_1-Pad1) -> V_INT
- J5 pad 10: unconnected-(J5-Pin_10-Pad10) -> GND
- J5 pad 2: unconnected-(J5-Pin_2-Pad2) -> CELL_GPIO4
- J5 pad 3: unconnected-(J5-Pin_3-Pad3) -> CELL_GPIO2
- J5 pad 4: unconnected-(J5-Pin_4-Pad4) -> CELL_GPIO1
- J5 pad 5: unconnected-(J5-Pin_5-Pad5) -> SDA
- J5 pad 6: unconnected-(J5-Pin_6-Pad6) -> SCL
- J5 pad 7: unconnected-(J5-Pin_7-Pad7) -> RI
- J5 pad 8: unconnected-(J5-Pin_8-Pad8) -> RTS
- J5 pad 9: unconnected-(J5-Pin_9-Pad9) -> CTS
- J9 pad 1: unconnected-(J9-Pin_1-Pad1) -> V_INT
- J9 pad 10: unconnected-(J9-Pin_10-Pad10) -> GND
- J9 pad 9: unconnected-(J9-Pin_9-Pad9) -> CELL_GPIO5

Commit message: test1
Parts:
- added R8: 10K 1%, Resistor_SMD:R_0402_1005Metric, F.Cu at (140.2, 82.5)
- added TP1: TestPoint_Small, TestPoint:TestPoint_Pad_1.0x1.0mm, F.Cu at (154.2, 84.5)
- moved L1 9.03 mm to (132.3, 99.7)
- moved R15 8.89 mm to (129.5, 107.1)
- moved R17 8.89 mm to (131.1, 106.4)
- moved R7 8.89 mm to (131.1, 110.6)
- moved C17 8.89 mm to (131.3, 109.6)
- moved C18 8.89 mm to (132.7, 104.6)
- moved C5 8.89 mm to (130.6, 104.8)
- moved LED1 8.89 mm to (129.5, 109.9)
- moved R16 8.89 mm to (131.1, 107.5)
- moved C6 8.89 mm to (131.1, 108.5)
- moved C11 8.26 mm to (134.3, 86.1)
- moved R14 8.26 mm to (137.3, 93.1)
- moved C12 8.26 mm to (134.3, 88.4)
- moved C15 8.26 mm to (134.2, 84.2)
- moved R12 8.26 mm to (134.2, 83.1)
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Connections:
- IC1 pad 6: CTS -> CELL_CTS
- IC1 pad 7: RTS -> CELL_RTS
- R1 pad 2: RTS -> CELL_RTS
- U4 pad 10: D6 -> ARDUINO_RTS
- U4 pad 12: unconnected-(U4-B2Y-Pad12) -> ARDUINO_CTS
- U4 pad 3: unconnected-(U4-A2-Pad3) -> CELL_CTS
- U4 pad 5: CELL_GPIO3 -> CELL_RTS

Commit message: test1
Parts:
- added C25: 100N 10V, Capacitor_SMD:C_0201_0603Metric, F.Cu at (145.5, 80.6)
- added C26: 100N 10V, Capacitor_SMD:C_0201_0603Metric, F.Cu at (154.8, 80.6)
- added JP6: SolderJumper_2_Open, Jumper:SolderJumper-2_P1.3mm_Open_RoundedPad1.0x1.5mm, B.Cu at (150.7, 94.0)
- added JP7: SolderJumper_2_Open, Jumper:SolderJumper-2_P1.3mm_Open_RoundedPad1.0x1.5mm, B.Cu at (150.7, 91.5)
- added JP8: SolderJumper_2_Open, Jumper:SolderJumper-2_P1.3mm_Open_RoundedPad1.0x1.5mm, B.Cu at (156.3, 92.7)
- added JP9: SolderJumper_2_Open, Jumper:SolderJumper-2_P1.3mm_Open_RoundedPad1.0x1.5mm, B.Cu at (156.3, 90.2)
- added R18: 0R0 0%, Resistor_SMD:R_0402_1005Metric, F.Cu at (145.6, 86.0)
- added R19: 10K 1%, Resistor_SMD:R_0402_1005Metric, F.Cu at (156.0, 85.4)
- added R9: 0R0 0%, Resistor_SMD:R_0402_1005Metric, F.Cu at (145.6, 86.9)
- added U1: TXU0204PWR, footprints2:TSSOP14_PW_TEX, F.Cu at (150.2, 82.9)
- JP1, JP2, JP3, JP4, JP5: moved to B.Cu
- moved JP3 16.5 mm to (134.6, 78.1)
- moved JP4 16.3 mm to (130.8, 77.0)
- moved R8 15.2 mm to (155.1, 85.4), turned to -90 degrees
- moved JP5 14.1 mm to (130.8, 74.5)
- moved JP2 12.2 mm to (138.6, 77.0)
- moved JP1 12.1 mm to (138.6, 74.5), turned to 180 degrees
- moved U2 11.2 mm to (134.5, 75.2)
- moved TP1 9.41 mm to (153.4, 75.1)
Connections:
- R8 pad 1: CELL_GPIO3 -> Net-(U1-OE)
- R8 pad 2: D6 -> V_INT
- U8 pad 1: D2 -> D7
