File: LEXI-ADAM UNO SHIELD ver.01.kicad_sch (KiCad schematic)
At the start: 28 parts, among them IC1 LEXI-R10801D-00B-00, J1 SSW-106-03-G-S, J2 SSW-110-03-G-S, J23 Conn_Coaxial, J3 SSW-108-03-G-S, J4 SSW-108-03-G-S, J7 Conn_Coaxial, SW1 B3FS-1000P, SW4 B3FS-1000P, U4 TXU0204PWR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

Commit message: test1
Parts:
- IC1: footprint LEXIR10801D00B00 -> footprints2:LEXIR10801D00B00
Connections:
- net RI: now reaches IC1.10 (RI)
- net DSR: now reaches IC1.11 (DSR)
- net SCL: now reaches IC1.12 (SCL)
- net SDA: now reaches IC1.13 (SDA)
- net CELL_GPIO1: now reaches IC1.14 (GPIO1)
- net CELL_GPIO2: now reaches IC1.15 (GPIO2)
- net CELL_GPIO4: now reaches IC1.17 (GPIO4)
- net CELL_GPIO5: now reaches IC1.18 (GPIO5)
- net CELL_GPIO6: now reaches IC1.29 (GPIO6)
- net USB_BOOT: now reaches IC1.48 (USB_BOOT)
- net CTS: now reaches IC1.6 (CTS)
- net DCD: now reaches IC1.8 (DCD)

Commit message: test1
Parts:
- added R8: 10K 1%, Resistor_SMD:R_0402_1005Metric, symbol Resistors_with_manufacturer_PartNumber_2:10K_0402_1%
- added TP1: TestPoint_Small, TestPoint:TestPoint_Pad_1.0x1.0mm, symbol Connector:TestPoint_Small
- added TP2: TestPoint_Small, symbol Connector:TestPoint_Small
Connections:
- net CTS is gone; now on net CELL_CTS: IC1.6 (CTS)
- net CELL_GPIO3: now also R8.1; no longer U4.5 (A4Y)
- net D6: now also R8.2; no longer U4.10 (B4)
- net ARDUINO_CTS: now reaches U4.12 (B2Y)
- net ARDUINO_CTS: now also TP2.1
- net CELL_CTS: now reaches U4.3 (A2)
- net RTS renamed CELL_RTS
- net CELL_RTS: now also U4.5 (A4Y)
- new net ARDUINO_RTS: TP1.1, U4.10 (B4)
Other:
- note added: "STM32 should have USART1_RTS on PA12 and PB3 corresponding to D4(PA12)and D2(PB3)"
- moved on the sheet: R10, R11

Commit message: test1
Parts:
- added C25, C26: 100N 10V, Capacitor_SMD:C_0201_0603Metric, symbol Capacitors_with_manufacturer_PartNumber_2:CAP CER 0201 100N 10% 10V
- added JP6, JP7, JP8, JP9: SolderJumper_2_Open, Jumper:SolderJumper-2_P1.3mm_Open_RoundedPad1.0x1.5mm, symbol Jumper:SolderJumper_2_Open
- added R18, R9: 0R0 0%, Resistor_SMD:R_0402_1005Metric, symbol Resistors_with_manufacturer_PartNumber_2:0R0_0402_0%
- added R19: 10K 1%, Resistor_SMD:R_0402_1005Metric, symbol Resistors_with_manufacturer_PartNumber_2:10K_0402_1%
- added U1: TXU0204PWR, footprints2:TSSOP14_PW_TEX, symbol shield_design_library:TXU0204PWR
Connections:
- net ARDUINO_CTS: now also JP8.1 (A), JP9.1 (A)
- net ARDUINO_RTS: now also JP6.1 (A), JP7.1 (A)
- net CELL_GPIO3: now also U1.4 (A3Y); no longer R8.1
- net D2: now also JP6.2 (B); no longer U8.1 (1A)
- net D4: now also JP7.2 (B)
- net D5: now also JP8.2 (B)
- net D6: now also U1.11 (B3); no longer R8.2
- net D7: now also U8.1 (1A)
- net D8: now also JP9.2 (B)
- net GND: now also C25.2, C26.1, U1.7 (GND)
- net IOREF: now also C26.2, R18.1, R19.2, U1.14 (VCCB)
- net V_INT: now also R8.2, C25.1, R9.1, U1.1 (VCCA)
- net at C24.1, U8.5 (VCC): now also R18.2, R9.2
- new net: R19.1, R8.1, U1.8 (OE)
Other:
- note added: "STM32 has USART1_CTS on GPIOs PA11 and PB4 corresponding to ARDUINO D5 (PA11) and ARDUINO D8 (PB4)"
- note added: "STM32 has USART1_RTS on GPIOs PA12 and PB3 corresponding to ARDUINO D4(PA12) and ARDUINO D2(PB3)"
- note removed: "STM32 should have USART1_RTS on PA12 and PB3 corresponding to D4(PA12)and D2(PB3)"
- moved on the sheet: C1, C13, C14, C19, C20, C21, C22, C23, C24, C4, C7, J23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
